Commit message: Add transmission tag

File: oparm_description/urdf/oparm.urdf.xacro (robot description, xacro)
@@ -5,4 +5,17 @@
   <!-- Import Gazebo settings -->
   <xacro:include filename="$(find oparm_description)/urdf/oparm.gazebo.xacro"/>
+  <!-- Transmission macro -->
+  <xacro:macro name="SimpleTransmission" params="joint n">
+    <transmission name="tran${n}">
+      <type>transmission_interface/SimpleTransmission</type>
+      <joint name="${joint}">
+        <hardwareInterface>hardware_interface/EffortJointInterface</hardwareInterface>
+      </joint>
+      <actuator name="motor${n}">
+        <hardwareInterface>hardware_interface/EffortJointInterface</hardwareInterface>
+        <mechanicalReduction>1</mechanicalReduction>
+      </actuator>
+    </transmission>
+  </xacro:macro>
   <!-- World -->
   <link name="world">
@@ -45,4 +58,6 @@
     <limit effort="1" velocity="1" lower="${-pi}" upper="${pi}"/>
   </joint>
+  <!-- Transmission 1 -->
+  <xacro:SimpleTransmission n="1" joint="joint1"/>
   <!-- Link 1 -->
   <link name="link1">
@@ -76,4 +91,6 @@
     <limit effort="1" velocity="1" lower="-1.57" upper="1.57"/>
   </joint>
+  <!-- Transmission 2 -->
+  <xacro:SimpleTransmission n="2" joint="joint2"/>
   <!-- Link 2 -->
   <link name="link2">
@@ -107,4 +124,6 @@
     <limit effort="1" velocity="1" lower="-1.75" upper="1.75"/>
   </joint>
+  <!-- Transmission 3 -->
+  <xacro:SimpleTransmission n="3" joint="joint3"/>
   <!-- Link 3 -->
   <link name="link3">
@@ -138,4 +157,6 @@
     <limit effort="1" velocity="1" lower="${-pi}" upper="${pi}"/>
   </joint>
+  <!-- Transmission 4 -->
+  <xacro:SimpleTransmission n="4" joint="joint4"/>
   <!-- Link 4 -->
   <link name="link4">
@@ -169,4 +190,6 @@
     <limit effort="1" velocity="1" lower="-1.57" upper="1.57"/>
   </joint>
+  <!-- Transmission 5 -->
+  <xacro:SimpleTransmission n="5" joint="joint5"/>
   <!-- Link 5 -->
   <link name="link5">

Commit message: Modify some inertia value in URDF

File: oparm_description/urdf/oparm.urdf.xacro (robot description, xacro)
@@ -78,7 +78,7 @@
       <origin xyz="0.0 0.0 3.9684358e-02"/>
       <mass value="4.2165803e-01"/>
-      <inertia ixx="5.7833699e-04" ixy="0.0" ixz="0.0"
-               iyy="4.3337111e-04" iyz="0.0"
-               izz="3.1986899e-04"/>
+      <inertia ixx="3.1986899e-04" ixy="0.0" ixz="0.0"
+               iyy="5.7833699e-04" iyz="0.0"
+               izz="4.3337111e-04"/>
     </inertial>
   </link>
@@ -113,5 +113,5 @@
       <inertia ixx="3.1351289e-03" ixy="0.0" ixz="0.0"
                iyy="3.8828211e-03" iyz="0.0"
-               izz="1.0956725e-03"/>
+               izz="-1.0956725e-03"/>
     </inertial>
   </link>
@@ -212,5 +212,5 @@
       <inertia ixx="6.6737478e-05" ixy="0.0" ixz="0.0"
                iyy="6.7027298e-05" iyz="0.0"
-               izz="3.9548898e-05"/>
+               izz="-3.9548898e-05"/>
     </inertial>
   </link>

Commit message: Add 'pi' property value

File: oparm_description/urdf/oparm.urdf.xacro (robot description, xacro)
@@ -5,4 +5,6 @@
   <!-- Import Gazebo settings -->
   <xacro:include filename="$(find oparm_description)/urdf/oparm.gazebo.xacro"/>
+	<!-- Properties -->
+	<xacro:property name="pi" value="3.1415926"/>
   <!-- Transmission macro -->
   <xacro:macro name="SimpleTransmission" params="joint n">

Commit message: Modify effort and velocity value

File: oparm_description/urdf/oparm.urdf.xacro (robot description, xacro)
@@ -53,4 +53,5 @@
   </link>
   <!-- Joint 1 -->
+	<!-- ROBOTIS Dynamixel MX-106 -->
   <joint name="joint1" type="revolute">
     <parent link="base"/>
@@ -58,5 +59,5 @@
     <origin xyz="0 0 0.0085" rpy="0 0 0"/>
     <axis xyz="0 0 1"/>
-    <limit effort="1" velocity="1" lower="${-pi}" upper="${pi}"/>
+    <limit effort="8.4" velocity="0.212" lower="${-pi}" upper="${pi}"/>
   </joint>
   <!-- Transmission 1 -->
@@ -86,4 +87,5 @@
   </link>
   <!-- Joint 2 -->
+	<!-- ROBOTIS Dynamixel MX-106 (x2) -->
   <joint name="joint2" type="revolute">
     <parent link="link1"/>
@@ -91,5 +93,5 @@
     <origin xyz="0 0 0.06" rpy="0 0 0"/>
     <axis xyz="1 0 0"/>
-    <limit effort="1" velocity="1" lower="-1.57" upper="1.57"/>
+    <limit effort="16.8" velocity="0.118" lower="-1.57" upper="1.57"/>
   </joint>
   <!-- Transmission 2 -->
@@ -119,4 +121,5 @@
   </link>
   <!-- Joint 3 -->
+	<!-- ROBOTIS Dynamixel MX-106 -->
   <joint name="joint3" type="revolute">
     <parent link="link2"/>
@@ -124,5 +127,5 @@
     <origin xyz="0 0 0.215" rpy="0 0 0"/>
     <axis xyz="1 0 0"/>
-    <limit effort="1" velocity="1" lower="-1.75" upper="1.75"/>
+    <limit effort="8.4" velocity="0.118" lower="-1.75" upper="1.75"/>
   </joint>
   <!-- Transmission 3 -->
@@ -152,4 +155,5 @@
   </link>
   <!-- Joint 4 -->
+	<!-- ROBOTIS Dynamixel MX-28 -->
   <joint name="joint4" type="revolute">
     <parent link="link3"/>
@@ -157,5 +161,5 @@
     <origin xyz="0 0 0.085" rpy="0 0 0"/>
     <axis xyz="0 0 1"/>
-    <limit effort="1" velocity="1" lower="${-pi}" upper="${pi}"/>
+    <limit effort="2.5" velocity="0.276" lower="${-pi}" upper="${pi}"/>
   </joint>
   <!-- Transmission 4 -->
@@ -185,4 +189,5 @@
   </link>
   <!-- Joint 5-->
+	<!-- ROBOTIS Dynamixel MX-28 -->
   <joint name="joint5" type="revolute">
     <parent link="link4"/>
@@ -190,5 +195,5 @@
     <origin xyz="0 0 0.0725" rpy="0 0 0"/>
     <axis xyz="1 0 0"/>
-    <limit effort="1" velocity="1" lower="-1.57" upper="1.57"/>
+    <limit effort="2.5" velocity="0.118" lower="-1.57" upper="1.57"/>
   </joint>
   <!-- Transmission 5 -->
